File: hardware/system/system.kicad_sch (KiCad schematic)
At the start: 44 parts, among them SW1 SW_Reed, SW2 SW_Push, SW3 SW_Reed, SW4 SW_Reed, U1 NE555P, U2 NE555P, U3 NE555P, U5 RED Strip, U7 RED Strip, U9 GREEN Strip

Commit message: style: save updated files to new version
Parts:
- U4, U6, U8: value ~ -> (none)
Connections:
- net at U7. (B): no longer U6. (GND)
- net at U9. (B): no longer U8. (GND)
- net at U5. (B): now also U4. (GND)
- new net: U6. (GND), U7. (B) (x2)
- new net: U8. (GND), U9. (B) (x2)
- new net: U4. (GND), U5. (B)
- now unconnected: U7. (B), U9. (B)
